File: Hardware/SarsatJRX-TH/SarsatJRX.kicad_sch (KiCad schematic)
At the start: 45 parts, among them J1 Conn_01x04_Pin, J2 Conn_Coaxial, J3 LilyPi GPIO Header, J4 Conn_01x04_Pin, U1 TLC2274, U2 TLC2274, U3 SA818S-U

Commit message: Added schematics.
Other:
- company: (none) -> F4JRX - ADRASEC 31
- title: (none) -> SarsatJRX signal board
